File: PCB/RP2040_Count.kicad_sch (KiCad schematic)
At the start: 17 parts, among them J2 String1, J3 OLED, SW1 Test, U2 AMS1117-5.0, U4 74AHCT1G125, U4 INA219BxD, U5 RP2040-Tiny

Commit message: added BOM
Parts:
- C5: Digi-Key_PN (none) -> 1276-1005-1-ND; MPN (none) -> CL10B104KO8NNNC
- C6: Digi-Key_PN (none) -> 1276-1005-1-ND; LCSC (none) -> C14663; LCSC_PN (none) -> C14663; MPN (none) -> CL10B104KO8NNNC
- J3: Digi-Key_PN S7002-ND -> (none); LCSC C225501 -> (none); MPN PPTC041LFBN-RC -> (none)
- R2: Digi-Key_PN (none) -> CSRN2512FTR100CT-ND; LCSC (none) -> C2903476; MPN (none) -> CSRN2512FTR100
- R3, R4: Digi-Key_PN (none) -> 311-10.0KHRCT-ND; LCSC (none) -> C25804; MPN (none) -> RC0603FR-0710KL
- SW1: Digi-Key_PN (none) -> CKN10880CT-ND; MPN (none) -> PTS645SL43SMTR92 LFS
- U4: Digi-Key_PN (none) -> 296-27899-1-ND; LCSC PN C138706 -> (none); LCSC_PN (none) -> C138706; MPN (none) -> INA219BIDR
Changed lines of the file:
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@@
+			)
+		)
+		(property "Digi-Key_PN" "1276-1005-1-ND"
+			(at 124.46 41.275 0)
+			(effects
+				(font
+					(size 1.27 1.27)
+				)
+				(hide yes)
+			)
+		)
+		(property "MPN" "CL10B104KO8NNNC"
+			(at 124.46 41.275 0)
+			(effects
+				(font
+					(size 1.27 1.27)
+				)
+				(hide yes)
 			)
 		)
@@
 			)
 		)
+		(property "Digi-Key_PN" "311-10.0KHRCT-ND"
+			(at 126.365 65.405 0)
+			(effects
+				(font
+					(size 1.27 1.27)
+				)
+				(hide yes)
+			)
+		)
+		(property "LCSC" "C25804"
+			(at 126.365 65.405 0)
+			(effects
+				(font
+					(size 1.27 1.27)
+				)
+				(hide yes)
+			)
+		)
+		(property "MPN" "RC0603FR-0710KL"
+			(at 126.365 65.405 0)
+			(effects
+				(font
+					(size 1.27 1.27)
+				)
+				(hide yes)
+			)
+		)
 		(pin "1"
 		)
@@
 			)
 		)
-		(property "Datasheet" ""
+		(property "Datasheet" "https://www.amazon.com/Waveshare-RP2040-Tiny-Development-Raspberry-Microcontroller/dp/B0C4FC84V9"
 			(at 158.75 105.41 0)
 			(effects
@@
 			)
 		)
+		(property "Digi-Key_PN" "1276-1005-1-ND"
+			(at 149.86 107.95 0)
+			(effects
+				(font
+					(size 1.27 1.27)
+				)
+				(hide yes)
+			)
+		)
+		(property "LCSC" "C14663"
+			(at 149.86 107.95 0)
+			(effects
+				(font
+					(size 1.27 1.27)
+				)
+				(hide yes)
+			)
+		)
+		(property "LCSC_PN" "C14663"
+			(at 149.86 107.95 0)
+			(effects
+				(font
+					(size 1.27 1.27)
+				)
+				(hide yes)
+			)
+		)
+		(property "MPN" "CL10B104KO8NNNC"
+			(at 149.86 107.95 0)
+			(effects
+				(font
+					(size 1.27 1.27)
+				)
+				(hide yes)
+			)
+		)
 		(pin "1"
 		)
@@
 			)
 		)
+		(property "Digi-Key_PN" "311-10.0KHRCT-ND"
+			(at 132.715 65.405 0)
+			(effects
+				(font
+					(size 1.27 1.27)
+				)
+				(hide yes)
+			)
+		)
+		(property "LCSC" "C25804"
+			(at 132.715 65.405 0)
+			(effects
+				(font
+					(size 1.27 1.27)
+				)
+				(hide yes)
+			)
+		)
+		(property "MPN" "RC0603FR-0710KL"
+			(at 132.715 65.405 0)
+			(effects
+				(font
+					(size 1.27 1.27)
+				)
+				(hide yes)
+			)
+		)
 		(pin "1"
 		)
@@
 			)
 		)
-		(property "Datasheet" "~"
+		(property "Datasheet" "https://www.amazon.com/dp/B06XRBTBTB/ref=sspa_dk_detail_0"
 			(at 232.41 102.87 0)
 			(effects
@@
 			)
 		)
-		(property "Digi-Key_PN" "S7002-ND"
+		(property "Digi-Key_PN" ""
 			(at 232.41 102.87 0)
 			(effects
@@
 			)
 		)
-		(property "MPN" "PPTC041LFBN-RC"
+		(property "MPN" ""
 			(at 232.41 102.87 0)
 			(effects
@@
 			)
 		)
-		(property "LCSC" "C225501"
+		(property "LCSC" ""
 			(at 232.41 102.87 0)
 			(effects
@@
 			)
 		)
+		(property "Digi-Key_PN" "CKN10880CT-ND"
+			(at 238.125 125.095 0)
+			(effects
+				(font
+					(size 1.27 1.27)
+				)
+				(hide yes)
+			)
+		)
+		(property "MPN" "PTS645SL43SMTR92 LFS"
+			(at 238.125 125.095 0)
+			(effects
+				(font
+					(size 1.27 1.27)
+				)
+				(hide yes)
+			)
+		)
 		(pin "1"
 		)
@@
 			)
 		)
+		(property "Digi-Key_PN" "1276-1005-1-ND"
+			(at 203.2 39.37 0)
+			(effects
+				(font
+					(size 1.27 1.27)
+				)
+				(hide yes)
+			)
+		)
+		(property "MPN" "CL10B104KO8NNNC"
+			(at 203.2 39.37 0)
+			(effects
+				(font
+					(size 1.27 1.27)
+				)
+				(hide yes)
+			)
+		)
 		(pin "1"
 		)
@@
 			)
 		)
-		(property "LCSC PN" "C138706"
+		(property "LCSC PN" ""
 			(at 116.205 57.785 0)
 			(effects
@@
 					(size 1.27 1.27)
 				)
+			)
+		)
+		(property "Digi-Key_PN" "296-27899-1-ND"
+			(at 116.205 57.785 0)
+			(effects
+				(font
+					(size 1.27 1.27)
+				)
+				(hide yes)
+			)
+		)
+		(property "LCSC_PN" "C138706"
+			(at 116.205 57.785 0)
+			(effects
+				(font
+					(size 1.27 1.27)
+				)
+				(hide yes)
+			)
+		)
+		(property "MPN" "INA219BIDR"
+			(at 116.205 57.785 0)
+			(effects
+				(font
+					(size 1.27 1.27)
+				)
+				(hide yes)
 			)
 		)
@@
 			(at 97.155 57.785 0)
 			(effects
+				(font
+					(size 1.27 1.27)
+				)
+				(hide yes)
+			)
+		)
+		(property "Digi-Key_PN" "CSRN2512FTR100CT-ND"
+			(at 97.155 57.785 0)
+			(effects
+				(font
+					(size 1.27 1.27)
+				)
+				(hide yes)
+			)
+		)
+		(property "LCSC" "C2903476"
+			(at 97.155 57.785 0)
+			(effects
+				(font
+					(size 1.27 1.27)
+				)
+				(hide yes)
+			)
+		)
+		(property "MPN" "CSRN2512FTR100"
+			(at 97.155 57.785 0)
+			(effects

Commit message: rename to v1
Parts:
- J3: LCSC (none) -> C225501
- R2: LCSC C2903476 -> C23140
- TB1: LCSC_PN (none) -> C23140
- U4: LCSC C7484 -> C138706; LCSC_PN C7484 -> C138706
Changed lines of the file:
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@@
 		(title "RP2040 Count")
 		(date "2024-02-11")
-		(rev "v2")
+		(rev "v1")
 	)
 	(junction
@@
 	(label "DOUT1"
 		(at 213.995 55.88 0)
-		(fields_autoplaced yes)
 		(effects
 			(font
@@
 	(label "PWR"
 		(at 49.53 118.11 0)
-		(fields_autoplaced yes)
 		(effects
 			(font
@@
 			)
 		)
-		(property "LCSC_PN" "C7484"
+		(property "LCSC_PN" "C138706"
 			(at 200.025 55.88 0)
 			(effects
@@
 			)
 		)
-		(property "LCSC" "C7484"
+		(property "LCSC" "C138706"
 			(at 200.025 55.88 0)
 			(effects
@@
 			)
 		)
-		(property "LCSC" ""
+		(property "LCSC" "C225501"
 			(at 232.41 102.87 0)
 			(effects
@@
 			)
 		)
-		(property "LCSC_PN" ""
+		(property "LCSC_PN" "C23140"
 			(at 31.115 88.265 0)
 			(effects
@@
 			)
 		)
-		(property "LCSC" "C2903476"
+		(property "LCSC" "C23140"
 			(at 97.155 57.785 0)
 			(effects
