File: V2 Lite/PCB/RP2040_Count.kicad_pcb (KiCad board)
At the start: 2 copper layers, 53.5 x 26.5 mm, 21 parts, among them J1 PRMG, J2 String1, J3 OLED, SW1 Test, U1 74AHCT1G125, U2 AP2112K-3.3, U3 AMS1117-5.0, U4 INA219BxD, U6 ATtiny1614-SS

Commit message: working on new versions
Parts:
- added D1: 3v3, LED_SMD:LED_0603_1608Metric, F.Cu at (142.8, 80.6)
- added R5: 330, Resistor_SMD:R_0603_1608Metric_Pad0.98x0.95mm_HandSolder, F.Cu at (142.8, 77.2)
- G***: footprint Scotts:chewi_15 -> Scotts:chewi_10
- moved G*** 1.20 mm to (148.6, 77.7), turned to 0 degrees
Routing:
- net Net-(D1-K): track 0.00 -> 1.70 mm
- net +3.3V: track 45.8 -> 46.9 mm
- net GND: vias 101 -> 102
Other:
- board text added: "${TITLE} ${REVISION} ${COMPANY}"
- board text removed: "${TITLE} ${REVISION}"
