File: V2 Lite/PCB/RP2040_Count.kicad_sch (KiCad schematic)
At the start: 20 parts, among them J1 PRMG, J2 String1, J3 OLED, SW1 Test, U1 74AHCT1G125, U2 AP2112K-3.3, U3 AMS1117-5.0, U4 INA219BxD, U6 ATtiny1614-SS

Commit message: working on new versions
Parts:
- added D1: 3v3, LED_SMD:LED_0603_1608Metric, symbol Device:LED_Filled
- added R5: 330, Resistor_SMD:R_0603_1608Metric_Pad0.98x0.95mm_HandSolder, symbol Device:R
Connections:
- net +3.3V: now also D1.2 (A)
- net GND: now also R5.2
- new net: D1.1 (K), R5.1
Other:
- company: (none) -> S&B Designs LLC
- title: RP2040 Count Lite -> SB Pixel Count Lite
