File: V2 Lite/PCB/SB_Pixel_Count.kicad_sch (KiCad schematic)
At the start: 17 parts, among them J2 String1, J3 OLED, SW1 Test, U2 AMS1117-5.0, U2 MOUDLE-SEEEDUINO-XIAO, U4 74AHCT1G125, U4 INA219BxD

Commit message: Rename RP2040_Count files/folders to SB_Pixel_Count across all variants
Renames the KiCad project quads (.kicad_pcb/.kicad_sch/.kicad_pro/.kicad_prl),
exported BOM/gerber/production files, case STL/FCStd files, and the
Firmware/RP2040_Count sketch (-> Firmware/SB_Pixel_Count, matching the
required folder/.ino name convention) in V1, V2, V2 Lite, and V3 Pro.

Fixes up internal cross-references that would otherwise go stale:
- kicad_pcb sheetfile metadata and kicad_sch symbol instance "project" fields
- kicad_pro/kicad_prl self-referencing "filename" fields and bom_export_filename
- .github/workflows/compile.yml and drc.yml sketch/DRC paths
- README.md links and ATtiny1614_Count.ino header comments

Verified the renamed Firmware/SB_Pixel_Count sketch still compiles
(VERSION2/seeed_xiao_rp2040) after the rename.

Co-Authored-By: Claude Sonnet 5 <noreply@anthropic.com>
Parts:
- removed U2: MOUDLE-SEEEDUINO-XIAO, XIAO_PCB:MOUDLE14P-2.54-21X17.8MM_scott, symbol MOUDLE-SEEEDUINO-XIAO:MOUDLE-SEEEDUINO-XIAO
- added C2: 10uF, Capacitor_SMD:C_0805_2012Metric_Pad1.18x1.45mm_HandSolder, symbol Device:CP
- added D1: 3v3, LED_SMD:LED_0603_1608Metric, symbol Device:LED_Filled
- added J1: PRMG, Connector_PinHeader_2.54mm:PinHeader_1x03_P2.54mm_Vertical, symbol Connector_Generic:Conn_01x03
- added R5: 330, Resistor_SMD:R_0603_1608Metric_Pad0.98x0.95mm_HandSolder, symbol Device:R
- added U2: AP2112K-3.3, Package_TO_SOT_SMD:SOT-23-5, symbol Regulator_Linear:AP2112K-3.3
- added U6: ATtiny1614-SS, Package_SO:SOIC-14_3.9x8.7mm_P1.27mm, symbol MCU_Microchip_ATtiny:ATtiny1614-SS
- renumbered C5 to C1, C2 to C3, C3 to C4, R7 to R1, U4 to U1, U2 to U3
Connections:
- net +3.3V: now also C6.2, C2.1, D1.2 (A), J1.1 (Pin_1), U2.5 (VOUT), U6.1 (VCC)
- net +5V: now also U2.1 (VIN), U2.3 (EN); no longer C6.2
- net GND: now also C2.2, J1.3 (Pin_3), R5.2, U2.2 (GND), U6.14 (GND)
- net I2C_SCL: now also U6.9 (PB0)
- net I2C_SDA: now also U6.8 (PB1)
- net OUT1: now also U6.2 (PA4)
- net SW1: now also U6.3 (PA5)
- new net: D1.1 (K), R5.1
- new net UPDI: J1.2 (Pin_2), U6.10 (~{RESET}/PA0)
Other:
- company: (none) -> S&B Designs LLC
- title: SB Pixel Count -> SB Pixel Count Lite
- moved on the sheet: C6
