File: V2/PCB/SB_Pixel_Count.kicad_pcb (KiCad board)
At the start: 2 copper layers, 53.5 x 26.5 mm, 18 parts, among them J2 String1, J3 OLED, SW1 Test, U1 74AHCT1G125, U2 MOUDLE-SEEEDUINO-XIAO, U3 AMS1117-5.0, U4 INA219BxD

Commit message: Add company name to title blocks; fix V3 Pro SW1/SW2 push-button DRC
Add (company "S&B Designs LLC") to V1/V2/V3 Pro's PCB and schematic
title blocks, matching V2 Lite, and add \${COMPANY} to each board's
silkscreen gr_text so it's printed on the physical board too.

Also includes KiCad-side board edits made while investigating the
SW1/SW2 "unconnected pad" DRC warnings on V3 Pro: added
lib/Scotts.pretty/SW_PUSH_6mm.kicad_mod, a copy of the standard
4-leg tactile switch footprint with unique pad numbers (1-4) instead
of the original's duplicated 1/1/2/2 numbering. The two redundant
mechanical-only legs (pads 3/4) are left with no net assigned, so
DRC's missing-connection check no longer applies to them. V3 Pro's
SW1/SW2 now use this footprint. Regenerated gerbers/BOM/fp-info-cache
reflect the resave.

Co-Authored-By: Claude Sonnet 5 <noreply@anthropic.com>
Other:
- board text added: "${TITLE} ${REVISION} ${COMPANY}"
- board text removed: "${TITLE} ${REVISION}"
Changed lines of the file:
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@@
 		(date "2024-02-11")
 		(rev "v2")
+		(company "S&B Designs LLC")
 	)
 	(layers
@@
 		)
 	)
-	(gr_text "${TITLE} ${REVISION}"
+	(gr_text "${TITLE} ${REVISION}\n${COMPANY}"
 		(at 117.55 92.67 270)
 		(layer "B.SilkS")
