File: V2/PCB/SB_Pixel_Count.kicad_sch (KiCad schematic)
At the start: 22 parts, among them J1 PRMG, J2 String1, J3 OLED, SW1 Test, U1 74AHCT1G125, U2 AP2112K-3.3, U3 AMS1117-5.0, U4 INA219BxD, U6 ATtiny1614-SS

Commit message: Rename RP2040_Count files/folders to SB_Pixel_Count across all variants
Renames the KiCad project quads (.kicad_pcb/.kicad_sch/.kicad_pro/.kicad_prl),
exported BOM/gerber/production files, case STL/FCStd files, and the
Firmware/RP2040_Count sketch (-> Firmware/SB_Pixel_Count, matching the
required folder/.ino name convention) in V1, V2, V2 Lite, and V3 Pro.

Fixes up internal cross-references that would otherwise go stale:
- kicad_pcb sheetfile metadata and kicad_sch symbol instance "project" fields
- kicad_pro/kicad_prl self-referencing "filename" fields and bom_export_filename
- .github/workflows/compile.yml and drc.yml sketch/DRC paths
- README.md links and ATtiny1614_Count.ino header comments

Verified the renamed Firmware/SB_Pixel_Count sketch still compiles
(VERSION2/seeed_xiao_rp2040) after the rename.

Co-Authored-By: Claude Sonnet 5 <noreply@anthropic.com>
Parts:
- removed C2: 10uF, Capacitor_SMD:C_0805_2012Metric_Pad1.18x1.45mm_HandSolder, symbol Device:CP
- removed D1: 3v3, LED_SMD:LED_0603_1608Metric, symbol Device:LED_Filled
- removed J1: PRMG, Connector_PinHeader_2.54mm:PinHeader_1x03_P2.54mm_Vertical, symbol Connector_Generic:Conn_01x03
- removed R5: 330, Resistor_SMD:R_0603_1608Metric_Pad0.98x0.95mm_HandSolder, symbol Device:R
- removed U2: AP2112K-3.3, Package_TO_SOT_SMD:SOT-23-5, symbol Regulator_Linear:AP2112K-3.3
- removed U6: ATtiny1614-SS, Package_SO:SOIC-14_3.9x8.7mm_P1.27mm, symbol MCU_Microchip_ATtiny:ATtiny1614-SS
- added U2: MOUDLE-SEEEDUINO-XIAO, XIAO_PCB:MOUDLE14P-2.54-21X17.8MM_scott, symbol MOUDLE-SEEEDUINO-XIAO:MOUDLE-SEEEDUINO-XIAO
- renumbered C3 to C2, C4 to C3, C1 to C5, R1 to R7, U3 to U2, U1 to U4
Connections:
- net +3.3V: now also U2.12 (3V3); no longer C6.2
- net +5V: now also C6.2, U2.14 (5V)
- net GND: now also U2.13 (GND)
- net I2C_SCL: now also U2.6 (PA9_A5_D5_SCL)
- net I2C_SDA: now also U2.5 (PA8_A4_D4_SDA)
- net OUT1: now also U2.7 (PB08_A6_D6_TX)
- net SW1: now also U2.8 (PB09_A7_D7_RX)
Other:
- company: S&B Designs LLC -> (none)
- title: SB Pixel Count Lite -> SB Pixel Count
- moved on the sheet: C6

Commit message: Add company name to title blocks; fix V3 Pro SW1/SW2 push-button DRC
Add (company "S&B Designs LLC") to V1/V2/V3 Pro's PCB and schematic
title blocks, matching V2 Lite, and add \${COMPANY} to each board's
silkscreen gr_text so it's printed on the physical board too.

Also includes KiCad-side board edits made while investigating the
SW1/SW2 "unconnected pad" DRC warnings on V3 Pro: added
lib/Scotts.pretty/SW_PUSH_6mm.kicad_mod, a copy of the standard
4-leg tactile switch footprint with unique pad numbers (1-4) instead
of the original's duplicated 1/1/2/2 numbering. The two redundant
mechanical-only legs (pads 3/4) are left with no net assigned, so
DRC's missing-connection check no longer applies to them. V3 Pro's
SW1/SW2 now use this footprint. Regenerated gerbers/BOM/fp-info-cache
reflect the resave.

Co-Authored-By: Claude Sonnet 5 <noreply@anthropic.com>
Other:
- company: (none) -> S&B Designs LLC
Changed lines of the file:
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@@
 		(date "2024-02-11")
 		(rev "v2")
+		(company "S&B Designs LLC")
 	)
 	(junction
