File: V3 Pro/PCB/RP2040_Count.kicad_sch (KiCad schematic)
At the start: 19 parts, among them J2 String1, J3 OLED, SW1 Test, SW2 Test, U1 74AHCT1G125, U2 MOUDLE-SEEEDUINO-XIAO, U3 AMS1117-5.0, U4 INA219BxD, U5 TF-123-ARP9H17

Commit message: Rename PCB/schematic title blocks to SB Pixel Count
Match the naming already applied to V2 Lite: V1/V2 title blocks
become "SB Pixel Count", V3 Pro becomes "SB Pixel Count Pro". The
title text flows into the silkscreen via the \${TITLE} gr_text
variable, so this updates both the schematic and the PCB silkscreen.

Co-Authored-By: Claude Sonnet 5 <noreply@anthropic.com>
Other:
- title: RP2040 Count Pro -> SB Pixel Count Pro
Changed lines of the file:
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@@
 	(paper "A4")
 	(title_block
-		(title "RP2040 Count Pro")
+		(title "SB Pixel Count Pro")
 		(date "2025-10-06")
 		(rev "v1")
