File: V1/PCB/SB_Pixel_Count.kicad_pcb (KiCad board)
At the start: 2 copper layers, 59 x 29.5 mm, 18 parts, among them J2 String1, J3 OLED, SW1 Test, U1 74AHCT1G125, U3 AMS1117-5.0, U4 INA219BxD, U5 RP2040-Tiny

Commit message: Add company name to title blocks; fix V3 Pro SW1/SW2 push-button DRC
Add (company "S&B Designs LLC") to V1/V2/V3 Pro's PCB and schematic
title blocks, matching V2 Lite, and add \${COMPANY} to each board's
silkscreen gr_text so it's printed on the physical board too.

Also includes KiCad-side board edits made while investigating the
SW1/SW2 "unconnected pad" DRC warnings on V3 Pro: added
lib/Scotts.pretty/SW_PUSH_6mm.kicad_mod, a copy of the standard
4-leg tactile switch footprint with unique pad numbers (1-4) instead
of the original's duplicated 1/1/2/2 numbering. The two redundant
mechanical-only legs (pads 3/4) are left with no net assigned, so
DRC's missing-connection check no longer applies to them. V3 Pro's
SW1/SW2 now use this footprint. Regenerated gerbers/BOM/fp-info-cache
reflect the resave.

Co-Authored-By: Claude Sonnet 5 <noreply@anthropic.com>
Connections:
- R1 pad 2: Net-(R1-Pad2) -> unconnected-(R1-Pad2)
- U1 pad 1: GND -> unconnected-(U1-Pad1)
- U1 pad 2: OUT1 -> unconnected-(U1-Pad2)
- U1 pad 3: GND -> unconnected-(U1-GND-Pad3)
- U1 pad 4: Net-(R1-Pad2) -> /DOUT1
- U1 pad 5: +5V -> unconnected-(U1-VCC-Pad5)
Routing:
- net GND: track 39.7 -> 37.8 mm
- net unconnected-(U1-GND-Pad3): track 0.00 -> 1.88 mm
- net /DOUT1: track 5.99 -> 7.74 mm
- net Net-(R1-Pad2): track 1.76 -> 0.00 mm
Other:
- board text added: "${TITLE} ${REVISION} ${COMPANY}"
- board text removed: "${TITLE} ${REVISION}"
