File: V1/PCB/SB_Pixel_Count.kicad_pcb (KiCad board)
At the start: 2 copper layers, 59 x 29.5 mm, 18 parts, among them J2 String1, J3 OLED, SW1 Test, U1 74AHCT1G125, U3 AMS1117-5.0, U4 INA219BxD, U5 RP2040-Tiny

Commit message: v1 fixes
Parts:
- SW1: footprint Button_Switch_SMD:SW_Push_1P1T_NO_6x6mm_H9.5mm -> Scotts:SW_Push_1P1T_NO_6x6mm_H9.5mm
Connections:
- R1 pad 2: unconnected-(R1-Pad2) -> Net-(R1-Pad2)
- SW1 pad 3: (no net) -> unconnected-(SW1-Pad3)
- SW1 pad 4: (no net) -> GND
- U1 pad 1: unconnected-(U1-Pad1) -> GND
- U1 pad 2: unconnected-(U1-Pad2) -> OUT1
- U1 pad 3: unconnected-(U1-GND-Pad3) -> GND
- U1 pad 4: /DOUT1 -> Net-(R1-Pad2)
- U1 pad 5: unconnected-(U1-VCC-Pad5) -> +5V
Routing:
- net GND: track 37.8 -> 39.7 mm
- net unconnected-(U1-GND-Pad3): track 1.88 -> 0.00 mm
- net /DOUT1: track 7.74 -> 5.99 mm
- net Net-(R1-Pad2): track 0.00 -> 1.76 mm
